Commit message: ws

File: toy_robot/robot.urdf (robot description, URDF)
Before this commit: robot toy_rrr, 5 links, 4 joints
Links:
- removed link link3
- link base_link: geometry visual mesh filename=package://toy_robot/meshes/base.stl
- link end_effector: geometry visual mesh filename=package://toy_robot/meshes/tip.stl
- link link1: geometry visual mesh filename=package://toy_robot/meshes/link1.stl
- link link2: geometry visual mesh filename=package://toy_robot/meshes/link2.stl
Joints:
- removed joint joint3
- joint joint1: origin xyz=0 0 0.10 rpy=0 0 0 -> xyz=0 0 0.05 rpy=0 0 0
- joint joint2: origin xyz=0 0 0 rpy=1.5708 0 0 -> xyz=0.15 0 0 rpy=0 0 0
- joint tool: parent link3 -> link2
